File: KiCad/GR_Slide_Pot_Controller.kicad_pcb (KiCad board)
At the start: 2 copper layers, 90.5 x 27.7 mm, 44 parts, among them J1 Conn_01x03, J5 Conn_01x02, J6 Conn_01x03, J7 Conn_01x04, J8 Conn_01x04, J9 Conn_01x02, U3 ATtiny804-SS, U4 L293DD

Commit message: Add files via upload
Parts:
- C4, C6: footprint Capacitor_SMD:C_Elec_8x5.4 -> Capacitor_SMD:C_Elec_4x5.4
Routing:
- net +5V: track 81.4 -> 84.6 mm
