File: KiCad/GR_Slide_Pot_Controller.sch (KiCad schematic (older format))
At the start: 43 parts, among them J1 Conn_01x03, J5 Conn_01x02, J6 Conn_01x03, J7 Conn_01x04, J8 Conn_01x04, J9 Conn_01x02, U3 ATtiny804-SS, U4 L293DD

Commit message: Add files via upload
Parts:
- C4, C6: footprint Capacitor_SMD:C_Elec_8x5.4 -> Capacitor_SMD:C_Elec_4x5.4
- R7: symbol PSM60_Fader:PSM60-081A-103B2 -> GR_Slide_Pot_Controller-rescue:PSM60-081A-103B2-PSM60_Fader
- U4: symbol L293dd:L293DD -> GR_Slide_Pot_Controller-rescue:L293DD-L293dd
Changed lines of the file:
@@
 SCL
 $Comp
-L PSM60_Fader:PSM60-081A-103B2 R7
+L GR_Slide_Pot_Controller-rescue:PSM60-081A-103B2-PSM60_Fader R7
 U 1 1 6269F133
 P 6925 4825
@@
 $EndComp
 $Comp
-L L293dd:L293DD U4
+L GR_Slide_Pot_Controller-rescue:L293DD-L293dd U4
 U 1 1 626AC80A
 P 6625 1275
@@
 F 0 "C4" H 6516 3571 50  0000 L CNN
 F 1 "10uF 16v" H 6516 3480 50  0000 L CNN
-F 2 "Capacitor_SMD:C_Elec_8x5.4" H 6425 3525 50  0001 C CNN
+F 2 "Capacitor_SMD:C_Elec_4x5.4" H 6425 3525 50  0001 C CNN
 F 3 "~" H 6425 3525 50  0001 C CNN
 	1    6425 3525
@@
 F 0 "C6" H 9791 2071 50  0000 L CNN
 F 1 "10uF 16v" H 9791 1980 50  0000 L CNN
-F 2 "Capacitor_SMD:C_Elec_8x5.4" H 9700 2025 50  0001 C CNN
+F 2 "Capacitor_SMD:C_Elec_4x5.4" H 9700 2025 50  0001 C CNN
 F 3 "~" H 9700 2025 50  0001 C CNN
 	1    9700 2025
